Commit message: [Assets] update urdf

File: assets/Frame/frame.urdf (robot description, URDF)
Before this commit: robot frame, 2 links, 1 joints
Links:
- link frame_y: geometry collision mesh filename=package://hello_worlds/assets/Frame/frame.obj scale=1 1 1; visual mesh filename=package://hello_worlds/assets/Frame/frame.obj scale=1 1 1
- link frame_z: geometry collision mesh filename=package://hello_worlds/assets/Frame/frame.obj scale=1 1 1; visual mesh filename=package://hello_worlds/assets/Frame/frame_z.dae scale=1 1 1

File: assets/eve.urdf (robot description, URDF)
Before this commit: robot eve, 8 links, 7 joints
Links:
- link arm_left_link: geometry collision mesh filename=package://hello_worlds/assets/Eve/eve_arm_left.obj; visual mesh filename=package://hello_worlds/assets/Eve/eve_arm_left.obj
- link arm_right_link: geometry collision mesh filename=package://hello_worlds/assets/Eve/eve_arm_right.obj; visual mesh filename=package://hello_worlds/assets/Eve/eve_arm_right.obj
- link base_link: geometry collision mesh filename=package://hello_worlds/assets/Eve/eve_body.obj; visual mesh filename=package://hello_worlds/assets/Eve/eve_body.obj
- link eve_head: geometry collision mesh filename=package://hello_worlds/assets/Eve/eve_head.obj; visual mesh filename=package://hello_worlds/assets/Eve/eve_head.obj
