Commit message: [Asset] split adream ground floor windows

File: assets/Adream/adream.urdf (robot description, URDF)
Before this commit: robot adream, 17 links, 16 joints
Links:
- removed link adream_window_h20_1
- removed link adream_window_h20_2
- added link adream_window_door_1; visual mesh filename=package://hello_worlds/assets/Adream/windows/window_door.obj scale=1 1 1
- added link adream_window_door_2; visual mesh filename=package://hello_worlds/assets/Adream/windows/window_door.obj scale=1 1 1
- added link adream_window_door_outside_3x3_1; visual mesh filename=package://hello_worlds/assets/Adream/windows/window_door_ou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 scale=1 1 1
- added link adream_window_door_outside_3x3_2; visual mesh filename=package://hello_worlds/assets/Adream/windows/window_door_ou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 scale=1 1 1
- added link adream_window_door_outside_3x3_3; visual mesh filename=package://hello_worlds/assets/Adream/windows/window_door_ou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 scale=1 1 1
- added link adream_window_h20_4; visual mesh filename=package://hello_worlds/assets/Adream/windows/window_single_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 scale=1 1 1
- added link adream_window_h20_5; visual mesh filename=package://hello_worlds/assets/Adream/windows/window_single_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 scale=1 1 1
- added link adream_window_h20_6; visual mesh filename=package://hello_worlds/assets/Adream/windows/window_single_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 scale=1 1 1
- added link adream_window_h20_7; visual mesh filename=package://hello_worlds/assets/Adream/windows/window_four_fr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 scale=1 1 1
- added link adream_window_h20_8; visual mesh filename=package://hello_worlds/assets/Adream/windows/window_outside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 scale=1 1 1
- added link adream_window_h20_9; visual mesh filename=package://hello_worlds/assets/Adream/windows/window_outside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 scale=1 1 1
- added link adream_window_h22_1; visual mesh filename=package://hello_worlds/assets/Adream/windows/window_h22.obj scale=1 1 1
- added link adream_window_h22_2; visual mesh filename=package://hello_worlds/assets/Adream/windows/window_h22.obj scale=1 1 1
- added link adream_window_h22_3; visual mesh filename=package://hello_worlds/assets/Adream/windows/window_h22.obj scale=1 1.12 1
- added link adream_window_outside_3x3_1; visual mesh filename=package://hello_worlds/assets/Adream/windows/window_outside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 scale=1 1 1
- added link adream_window_outside_3x3_2; visual mesh filename=package://hello_worlds/assets/Adream/windows/window_outside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 scale=1 1 1
- link adream_window_h10_2: mass .0 -> None; geometry visual mesh filename=package://hello_worlds/assets/Adream/windows/window_outside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 scale=1 1.022 1
- link adream_window_h20_3: mass .0 -> None; geometry visual mesh filename=package://hello_worlds/assets/Adream/windows/window_single_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 scale=1 1 1
Joints:
- removed joint base_to_adream_window_h20_1
- removed joint base_to_adream_window_h20_2
- added joint base_to_adream_window_door_1: type fixed, parent adream_walls, child adream_window_door_1, origin xyz=-0.060789 6.0788 1.4258 rpy=0 0 0
- added joint base_to_adream_window_door_2: type fixed, parent adream_walls, child adream_window_door_2, origin xyz=-5.2078 8.2955 1.4258 rpy=0 0 0
- added joint base_to_adream_window_door_outside_3x3_1: type fixed, parent adream_walls, child adream_window_door_outside_3x3_1, origin xyz=11.573 15.98 1.5938 rpy=0 0 0
- added joint base_to_adream_window_door_outside_3x3_2: type fixed, parent adream_walls, child adream_window_door_outside_3x3_2, origin xyz=11.573 6.0135 1.5938 rpy=0 0 0
- added joint base_to_adream_window_door_outside_3x3_3: type fixed, parent adream_walls, child adream_window_door_outside_3x3_3, origin xyz=11.573 -3.9512 1.5938 rpy=0 0 0
- added joint base_to_adream_window_h20_4: type fixed, parent adream_walls, child adream_window_h20_4, origin xyz=8.8243 18.508 1.5531 rpy=0 0 0
- added joint base_to_adream_window_h20_5: type fixed, parent adream_walls, child adream_window_h20_5, origin xyz=7.584 18.508 1.5531 rpy=0 0 0
- added joint base_to_adream_window_h20_6: type fixed, parent adream_walls, child adream_window_h20_6, origin xyz=6.3587 18.508 1.5531 rpy=0 0 0
- added joint base_to_adream_window_h20_7: type fixed, parent adream_walls, child adream_window_h20_7
- added joint base_to_adream_window_h20_8: type fixed, parent adream_walls, child adream_window_h20_8, origin xyz=-0.060667 1.2035 1.8868 rpy=0 0 0
- added joint base_to_adream_window_h20_9: type fixed, parent adream_walls, child adream_window_h20_9, origin xyz=-0.060667 3.6972 1.8868 rpy=0 0 0
- added joint base_to_adream_window_h22_1: type fixed, parent adream_walls, child adream_window_h22_1, origin xyz=5.0627 -1.0579 1.7611 rpy=0 0 0
- added joint base_to_adream_window_h22_2: type fixed, parent adream_walls, child adream_window_h22_2, origin xyz=5.0627 -5.3393 1.7611 rpy=0 0 0
- added joint base_to_adream_window_h22_3: type fixed, parent adream_walls, child adream_window_h22_3, origin xyz=3.95 -0.04475 1.7611 rpy=0 0 0
- added joint base_to_adream_window_outside_3x3_1: type fixed, parent adream_walls, child adream_window_outside_3x3_1, origin xyz=11.573 1.0355 1.5932 rpy=0 0 0
- added joint base_to_adream_window_outside_3x3_2: type fixed, parent adream_walls, child adream_window_outside_3x3_2, origin xyz=11.571 11.001 1.5929 rpy=0 0 0
- joint base_to_adream_window_h10_2: origin (none) -> xyz=-2.8639 8.2988 1.4249 rpy=0 0 0
- joint base_to_adream_window_h20_3: origin (none) -> xyz=10.06 18.508 1.5531 rpy=0 0 0
